File: KiCad/X4CMoscatel.kicad_pcb (KiCad board)
At the start: 2 copper layers, 55 x 55 mm, 27 parts, among them J1 Conn_01x04, J2 Micro_SD_Card_Det_Hirose_DM3AT, J3 USB_C_Receptacle_USB2.0_14P, J4 Conn_01x02_Pin, J5 Conn_01x10_Pin, SW1 SW_Push, SW2 SW_Push, SW3 SW_Wuerth_450301014042, U1 ESP32-S3-WROOM-1, U3 LD1117V33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

Commit message: Upgrade tocho
Parts:
- added C1: 100nF, Capacitor_SMD:C_0805_2012Metric, F.Cu at (209.0, 98.5)
- added C5: 100nF, Capacitor_SMD:C_0805_2012Metric, F.Cu at (208.5, 95.5)
- added D4: BAT54S, Package_TO_SOT_SMD:SOT-23, F.Cu at (204.5, 91.1)
- added J6: Conn_01x02_Pin, Connector_PinSocket_2.54mm:PinSocket_1x02_P2.54mm_Vertical, F.Cu at (213.0, 94.0)
- added R10: 1M, Resistor_SMD:R_0805_2012Metric, F.Cu at (209.1, 91.5)
- added R8: 1M, Resistor_SMD:R_0805_2012Metric, F.Cu at (209.0, 101.5)
- added R9: 1M, Resistor_SMD:R_0805_2012Metric, F.Cu at (204.1, 101.5)
- added U2: MCP6002-xMC, Package_DFN_QFN:DFN-8-1EP_3x2mm_P0.5mm_EP1.75x1.45mm, F.Cu at (203.0, 97.5)
- moved SW3 17.3 mm to (195.0, 99.0)
- moved J2 0.65 mm to (166.0, 107.1)
Connections:
- U1 pad 5: unconnected-(U1-IO5-Pad5) -> /Piezoeléctrico/GPIO5
Routing:
- net /Piezoeléctrico/GPIO5: track 0.00 -> 40.2 mm, vias 0 -> 2
- net Net-(D1-K): track 44.0 -> 26.9 mm
- net Net-(U2A-+): track 0.00 -> 16.4 mm
- net Net-(J6-Pin_2): track 0.00 -> 11.3 mm
- net Net-(J4-Pin_1): track 33.1 -> 22.3 mm
- net 3V3: track 30.5 -> 39.3 mm, vias 8 -> 11
- net GND: track 17.8 -> 23.2 mm
- net Net-(U2B--): track 0.00 -> 0.50 mm
Other:
- board size 55 x 55 mm -> 55 x 55.5 mm
