File: KiCad/X4CMoscatel.kicad_sch (KiCad schematic)
At the start: 10 parts, among them SW1 SW_Push, SW2 SW_Push, U1 ESP32-S3-WROOM-1

Commit message: Upgrade tocho
Connections:
- net Piezoeléctrico/GPIO5: now reaches U1.5 (IO5)
Other:
- added sheet Piezoeléctrico (piezoeléctrico.kicad_sch)
Changed lines of the file:
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@@
+	(wire
+		(pts
+			(xy 125.73 88.9) (xy 78.74 88.9)
+		)
+		(stroke
+			(width 0)
+			(type default)
+		)
+	)
 	(wire
 		(pts
@@
 				)
 			)
+		)
+	)
+	(sheet
+		(at 59.69 86.36)
+		(size 19.05 5.08)
+		(exclude_from_sim no)
+		(in_bom yes)
+		(on_board yes)
+		(dnp no)
+		(fields_autoplaced yes)
+		(stroke
+			(width 0.1524)
+			(type solid)
+		)
+		(fill
+			(color 0 0 0 0.0000)
+		)
+		(property "Sheetname" "Piezoeléctrico"
+			(at 59.69 85.6484 0)
+			(effects
+				(font
+					(size 1.27 1.27)
+				)
+				(justify left bottom)
+			)
+		)
+		(property "Sheetfile" "piezoeléctrico.kicad_sch"
+			(at 59.69 92.0246 0)
+			(effects
+				(font
+					(size 1.27 1.27)
+				)
+				(justify left top)
+			)
+		)
+		(pin "GPIO5" input
+			(at 78.74 88.9 0)
+			(effects
+				(font
+					(size 1.27 1.27)
+				)
+				(justify right)
+			)
+		)
+		(instances
+			(project "X4CMoscatel"
+				(path "/24687d0d-f043-49b3-9437-7388bda4ef16"
+					(page "6")
+				)
+			)
